Commit message: Update plane.urdf.xacro

File: my_robot_description/urdf/plane.urdf.xacro (robot description, xacro)
@@ -22,5 +22,5 @@
         <origin rpy="1.57 0 0" xyz="-0.6 0.5 0"/>
         <geometry>
-          <mesh filename="package://my_robot_description/meshes/basic_plane.STL" scale="0.01 0.01 0.01"/>
+          <mesh filename="package://my_robot_description/meshes/basic_plane_2.STL" scale="0.01 0.01 0.01"/>
         </geometry>
         <material name="weird"/>
